File: LEDFB.sch (EAGLE design)
At the start: 7 parts

Commit message: Added additional schematic pages and wired the LEDs
Parts:
- added BATT1: AAA, adafruit:AAA
- added C2: 10uF, adafruit:C-USC0805
- added R10, R2, R3, R4, R8, R9: (no value), adafruit:R-US_R0805
- added R5, R6, R7: 10, adafruit:R-US_R0805
- added S2: (no value), adafruit:EG1218S
- added U$2, U$3, U$4: MMBT3904FSCT-ND, GuShH:MMBT3904FSCT-ND
- added U$5, U$6: LED_PIRANHA_5MM, SparkFun-LED:LED_PIRANHA_5MM
Connections:
- new net GREEN_CTRL: R7.2
- new net N$10: U$3.E
- new net N$11: U$4.E
- new net N$12: R5.1, U$2.B
- new net N$13: R6.1, U$3.B
- new net N$14: R7.1, U$4.B
- new net N$15: R8.1, U$6.BLU
- new net N$16: R4.2, R8.2, U$3.C
- new net N$17: R10.2, R9.2
- new net N$18: R9.1, U$5.GRN
- new net N$19: R10.1, U$6.GRN
- new net N$20: BATT1.-, C2.1
- new net N$4: R2.1, U$5.RED
- new net N$5: R3.1, U$6.RED
- new net N$8: R2.2, R3.2, U$2.C
- new net N$9: R4.1, U$5.BLU
- net BLUE_CTRL: now also R6.2
- net GND: now also BATT1.+, C2.2, U$2.E
- net RED_CTRL: now also R5.2
- net VCC: now also U$5.C, U$6.C
