File: Schematic and Layout/LEDFB.sch (EAGLE design)
At the start: 25 parts, among them U1 TLV61225L

Commit message: Changed stuff
Parts:
- added C3: 10uF, adafruit:C-USC0805
- added R11, R12: 4.7k, adafruit:R-US_M0805
- added U$7: LQH3NPN4R7NJ0, inductor:LQH3NPN4R7NJ0
- added U2: ITG-37013X3MM, itg_3701:ITG-37013X3MM
- R10, R4, R8, R9: value (none) -> 60
- R2, R3: value (none) -> 300
- U1: value TLV61225L -> TLV61225M; device TLV61225:TLV61225L -> TLV61225:TLV61225M
Connections:
- removed net N$10: U$3.E
- removed net N$11: U$4.E
- new net INT: U$1.6, U2.INT
- new net N$21: S2.P, U1.EN
- new net N$22: U$7.P$2, U1.L
- new net SCL: R12.1, U$1.14, U2.SCL/SCLK
- new net SDA: R11.1, U$1.15, U2.SDA/SDI
- net GND: now also C3.2, S2.O, U$3.E, U$4.E, U1.GND, U2.AD0/SDO, U2.FSYNC, U2.GND, U2.GND_RSVD
- net GREEN_CTRL: now also U$1.12
- net N$17: now also U$4.C
- net N$20: now also S2.S, U$7.P$1, U1.VIN
- net VCC: now also C3.1, R11.2, R12.2, U1.FB, U1.VOUT, U2.CS, U2.VDD, U2.VDDIO
Other:
- moved on the sheet: JP3, S2, U1
